File: gridfins/buck.kicad_sch (KiCad schematic)
At the start: 30 parts, among them Q1 SSM3K15AMFV,L3F, U6 SiC437AED-T1

Commit message: PCB + schematic updates
Solved footprint error which prevented PCB from updating

Deleted old buck converter PCB design (old buck now replaced with 2 for servo and linear acc)

Moved Snubber and crossed out capacitor network to the backside of board

Unsure whether if the +10V routing is valid - currently connected via tracers, not planes (may be a problem for current)

Restructured old pcb which previously had planes associated with no nets (assigned nets to them)

If current design approved, will proceed to carry out the same design for the servo controlling buck converter.
Parts:
- R21: value 113k -> 157k
Connections:
- net VOUT_H_Bridge is gone; now on net +10V: R21.2, R38.2
Changed lines of the file:
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@@
 		)
 	)
-	(text_box "Remove this resistor for 7.4V mode"
+	(text_box "Remove this resistor for 10V mode"
 		(exclude_from_sim no)
 		(at 124.46 46.99 0)
@@
 		)
 	)
-	(label "VOUT_H_Bridge"
+	(label "VOUT"
 		(at 121.92 52.07 180)
 		(effects
@@
 			)
 		)
-		(property "Value" "113k"
+		(property "Value" "157k"
 			(at 121.92 63.4969 0)
 			(effects

Commit message: Handoff
implemented changes advised by Will. Still a bit unsure about how the EPAD should be connected to ground. The PCB design of both buck converters for servo and Hbridge(linear accuator) was completed - but still needs to be reviewed
Parts:
- R38: value 442k -> 0; now not fitted
Changed lines of the file:
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@@
 		(in_bom yes)
 		(on_board yes)
-		(dnp no)
+		(dnp yes)
 		(property "Reference" "R38"
 			(at 132.08 60.96 0)
@@
 			)
 		)
-		(property "Value" "442k"
+		(property "Value" "0"
 			(at 132.08 63.4969 0)
 			(effects
