File: gridfins/buck.kicad_sch (KiCad schematic)
At the start: 30 parts, among them Q1 SSM3K15AMFV,L3F, U6 SiC437AED-T1

Commit message: formatting
Parts:
- C510: renamed from C64; value 0.1uF -> 100nF
- R501: renamed from R20; value 10k -> 10kΩ
- R502: renamed from R21; value 157k -> 157kΩ
- R503: renamed from R22; value 10k -> 10kΩ
- R504: renamed from R23; value 2.2 -> 2.2Ω
- R505: renamed from R24; value 1k -> 1kΩ
- R506: renamed from R38; value 0 -> 0Ω
- R507: renamed from R39; value 200k -> 200kΩ
- R508: renamed from R42; value 100k -> 100kΩ
- R509: renamed from R56; value 10k -> 10kΩ
- R510: renamed from R57; value 5.1R -> 5.1Ω
- renumbered C38 to C501, C39 to C502, C40 to C503, C46 to C504, C47 to C505, C48 to C506, C49 to C507, C61 to C508, C62 to C509, C65 to C511, C66 to C512, C75 to C513, C76 to C514, C77 to C515, C78 to C516, C79 to C517, L4 to L501, Q1 to Q501, U6 to U501
Other:
- note removed: "SPM10065VT-3R3M-D"

Commit message: feat: Post Jack review
Changed buck inductors to be wuerth. Reduced board footprint. Incorporated review feedback
Parts:
- L501: footprint iclr:IND_SPM10065VT-3R3M-D -> iclr:WE-XHMI_7070
Connections:
- net +10V: now also L501.2; no longer L501.1
- net SW: now also L501.1; no longer L501.2
Other:
- moved on the sheet: L501
Changed lines of the file:
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@@
 	(symbol
 		(lib_id "Device:L")
-		(at 59.69 81.28 90)
+		(at 59.69 81.28 270)
+		(mirror x)
 		(unit 1)
 		(body_style 1)
@@
 		(in_pos_files yes)
 		(dnp no)
-		(fields_autoplaced yes)
 		(property "Reference" "L501"
 			(at 59.69 77.47 90)
@@
 			)
 		)
-		(property "Footprint" "iclr:IND_SPM10065VT-3R3M-D"
+		(property "Footprint" "iclr:WE-XHMI_7070"
 			(at 59.69 81.28 0)
 			(hide yes)
