File: gridfins/IMU.kicad_sch (KiCad schematic)
At the start: 10 parts, among them IC1 2536030320001, U8 MMC5983MA, U9 H3LIS331DLTR

Commit message: formatting
Parts:
- renumbered C12 to C901, C34 to C902, C36 to C903, C41 to C904, C42 to C905, C44 to C906, C50 to C907, U9 to U901, IC1 to U902, U8 to U903
Other:
- note removed: "MISO"
- note removed: "MOSI"
- note removed: "SCLK"
- moved on the sheet: C901, C902, C903, C904, C905, U901
