File: gridfins/LinearActuator.kicad_sch (KiCad schematic)
At the start: 12 parts, among them J8 1053131104, U7 DRV8834PWP

Commit message: feat: Massive changes, board almost ready for review
Parts:
- removed C18: 10uF, Capacitor_SMD:C_0402_1005Metric, symbol Device:C_Polarized_Small
- added C30: 10uF, Capacitor_SMD:C_0805_2012Metric, symbol Device:C_Small
- added R46, R47: 10k, Resistor_SMD:R_0402_1005Metric, symbol Device:R
- added TP12: TestPoint, TestPoint:TestPoint_Pad_D1.0mm, symbol Connector:TestPoint
- R43, R44: value 0.32 -> 0.5; footprint Resistor_SMD:R_0402_1005Metric -> Resistor_SMD:R_2512_6332Metric
Connections:
- net GND: now also U7.25 (EPAD), C30.2; no longer U7.15 (CONFIG), U7.EPAD
- net NSLEEP: now also R46.1
- net VINT: no longer U7.14 (M1)
- net VM: now also C30.1
- net AOUT1: now reaches U7.4 (AOUT1)
- net AOUT1: now also J8.4; no longer J8.1
- net AOUT2: now reaches U7.6 (AOUT2)
- net AOUT2: now also J8.3; no longer J8.2
- net BOUT2: now reaches U7.7 (BOUT2)
- net BOUT2: now also J8.2; no longer J8.3
- net BOUT1: now reaches U7.9 (BOUT1)
- net BOUT1: now also J8.1; no longer J8.4
- net Fault: now reaches U7.16 (NFAULT)
- new net: R47.1, TP12.1, U7.15 (CONFIG)
- new net +3V3: R46.2, R47.2
- new net M1: U7.14 (M1)
- no-connect marks 1 -> 0
Other:
- note added: "https://www.omc-stepperonline.com/nema-14-bipolar-1-8deg-18ncm-25-5oz-in-0-8a-5-4v-35x35x34mm-4-wires-14hs13-0804s Nema 14 Bipolar stepper"

Commit message: formatting
Parts:
- C1102: renamed from C19; value 0.01uF -> 10nF
- C1103: renamed from C56; value 0.01uF -> 10nF
- C1104: renamed from C28; value 0.1uF -> 100nF
- R1101: renamed from R47; value 10k -> 10kΩ
- R1102: renamed from R40; value 51K -> 51kΩ
- R1103: renamed from R41; value 51K -> 51kΩ
- R1104: renamed from R46; value 10k -> 10kΩ
- R1105: renamed from R43; value 0.5 -> 0.5Ω
- R1106: renamed from R44; value 0.5 -> 0.5Ω
- TP1101: renamed from TP12; now left out of the parts list
- renumbered C57 to C1101, C29 to C1105, C30 to C1106, J8 to J1101, U7 to U1101
Changed lines of the file:
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@@
 		(body_style 1)
 		(exclude_from_sim no)
-		(in_bom yes)
+		(in_bom no)
 		(on_board yes)
 		(in_pos_files yes)
 		(dnp no)
 		(fields_autoplaced yes)
-		(property "Reference" "TP12"
+		(property "Reference" "TP1101"
 			(at 72.39 92.2019 0)
 			(show_name no)
@@
 			(project "gridfins"
 				(path "/7db990e4-92e1-4f99-b4d2-435bbec1ba83/a2b9d01a-f05c-4fe0-bfaf-c74e95793a8f"
-					(reference "TP12")
+					(reference "TP1101")
 					(unit 1)
 				)
@@
 		(in_pos_files yes)
 		(dnp no)
-		(property "Reference" "J8"
+		(property "Reference" "J1101"
 			(at 236.22 124.46 0)
 			(show_name no)
@@
 			(project "gridfins"
 				(path "/7db990e4-92e1-4f99-b4d2-435bbec1ba83/a2b9d01a-f05c-4fe0-bfaf-c74e95793a8f"
-					(reference "J8")
+					(reference "J1101")
 					(unit 1)
 				)
@@
 		(in_pos_files yes)
 		(dnp no)
-		(property "Reference" "R43"
+		(property "Reference" "R1105"
 			(at 177.546 89.154 90)
 			(show_name no)
@@
 			)
 		)
-		(property "Value" "0.5"
+		(property "Value" "0.5Ω"
 			(at 177.8 90.932 90)
 			(show_name no)
@@
 			(project "gridfins"
 				(path "/7db990e4-92e1-4f99-b4d2-435bbec1ba83/a2b9d01a-f05c-4fe0-bfaf-c74e95793a8f"
-					(reference "R43")
+					(reference "R1105")
 					(unit 1)
 				)
@@
 		(in_pos_files yes)
 		(dnp no)
-		(property "Reference" "C28"
+		(property "Reference" "C1104"
 			(at 192.278 76.454 0)
 			(show_name no)
@@
 			)
 		)
-		(property "Value" "0.1uF"
+		(property "Value" "100nF"
 			(at 192.278 78.232 0)
 			(show_name no)
@@
 			(project "gridfins"
 				(path "/7db990e4-92e1-4f99-b4d2-435bbec1ba83/a2b9d01a-f05c-4fe0-bfaf-c74e95793a8f"
-					(reference "C28")
+					(reference "C1104")
 					(unit 1)
 				)
@@
 		(dnp no)
 		(fields_autoplaced yes)
-		(property "Reference" "#PWR091"
+		(property "Reference" "#PWR01101"
 			(at 55.88 93.98 0)
 			(hide yes)
@@
 			(project "gridfins"
 				(path "/7db990e4-92e1-4f99-b4d2-435bbec1ba83/a2b9d01a-f05c-4fe0-bfaf-c74e95793a8f"
-					(reference "#PWR091")
+					(reference "#PWR01101")
 					(unit 1)
 				)
@@
 		(dnp no)
 		(fields_autoplaced yes)
-		(property "Reference" "#PWR092"
+		(property "Reference" "#PWR01102"
 			(at 59.69 82.55 0)
 			(hide yes)
@@
 			(project "gridfins"
 				(path "/7db990e4-92e1-4f99-b4d2-435bbec1ba83/a2b9d01a-f05c-4fe0-bfaf-c74e95793a8f"
-					(reference "#PWR092")
+					(reference "#PWR01102")
 					(unit 1)
 				)
@@
 		(in_pos_files yes)
 		(dnp no)
-		(property "Reference" "R40"
+		(property "Reference" "R1102"
 			(at 68.326 67.818 90)
 			(show_name no)
@@
 			)
 		)
-		(property "Value" "51K"
+		(property "Value" "51kΩ"
 			(at 68.072 77.216 90)
 			(show_name no)
@@
 			(project "gridfins"
 				(path "/7db990e4-92e1-4f99-b4d2-435bbec1ba83/a2b9d01a-f05c-4fe0-bfaf-c74e95793a8f"
-					(reference "R40")
+					(reference "R1102")
 					(unit 1)
 				)
@@
 		(in_pos_files yes)
 		(dnp no)
-		(property "Reference" "#PWR0113"
+		(property "Reference" "#PWR01107"
 			(at 187.96 106.68 0)
 			(hide yes)
@@
 			(project "gridfins"
 				(path "/7db990e4-92e1-4f99-b4d2-435bbec1ba83/a2b9d01a-f05c-4fe0-bfaf-c74e95793a8f"
-					(reference "#PWR0113")
+					(reference "#PWR01107")
 					(unit 1)
 				)
@@
 		(in_pos_files yes)
 		(dnp no)
-		(property "Reference" "#PWR016"
+		(property "Reference" "#PWR01105"
 			(at 184.15 76.2 0)
 			(hide yes)
@@
 			(project "gridfins"
 				(path "/7db990e4-92e1-4f99-b4d2-435bbec1ba83/a2b9d01a-f05c-4fe0-bfaf-c74e95793a8f"
-					(reference "#PWR016")
+					(reference "#PWR01105")
 					(unit 1)
 				)
@@
 		(dnp no)
 		(fields_autoplaced yes)
-		(property "Reference" "R47"
+		(property "Reference" "R1101"
 			(at 67.31 83.82 90)
 			(show_name no)
@@
 			)
 		)
-		(property "Value" "10k"
+		(property "Value" "10kΩ"
 			(at 67.31 86.36 90)
 			(show_name no)
@@
 			(project "gridfins"
 				(path "/7db990e4-92e1-4f99-b4d2-435bbec1ba83/a2b9d01a-f05c-4fe0-bfaf-c74e95793a8f"
-					(reference "R47")
+					(reference "R1101")
 					(unit 1)
 				)
@@
 		(dnp no)
 		(fields_autoplaced yes)
-		(property "Reference" "#PWR075"
+		(property "Reference" "#PWR01103"
 			(at 85.09 60.96 0)
 			(hide yes)
@@
 			(project "gridfins"
 				(path "/7db990e4-92e1-4f99-b4d2-435bbec1ba83/a2b9d01a-f05c-4fe0-bfaf-c74e95793a8f"
-					(reference "#PWR075")
+					(reference "#PWR01103")
 					(unit 1)
 				)
@@
 		(dnp no)
 		(fields_autoplaced yes)
-		(property "Reference" "U7"
+		(property "Reference" "U1101"
 			(at 127.781 59.69 0)
 			(show_name no)
@@
 			(project "gridfins"
 				(path "/7db990e4-92e1-4f99-b4d2-435bbec1ba83/a2b9d01a-f05c-4fe0-bfaf-c74e95793a8f"
-					(reference "U7")
+					(reference "U1101")
 					(unit 1)
 				)
@@
 		(in_pos_files yes)
 		(dnp no)
-		(property "Reference" "R41"
+		(property "Reference" "R1103"
 			(at 67.818 78.994 90)
 			(show_name no)
@@
 			)
 		)
-		(property "Value" "51K"
+		(property "Value" "51kΩ"
 			(at 68.58 70.104 90)
 			(show_name no)
@@
 			(project "gridfins"
 				(path "/7db990e4-92e1-4f99-b4d2-435bbec1ba83/a2b9d01a-f05c-4fe0-bfaf-c74e95793a8f"
-					(reference "R41")
+					(reference "R1103")
 					(unit 1)
 				)
@@
 		(in_pos_files yes)
 		(dnp no)
-		(property "Reference" "C29"
+		(property "Reference" "C1105"
 			(at 202.692 76.454 0)
 			(show_name no)
@@
 			(project "gridfins"
 				(path "/7db990e4-92e1-4f99-b4d2-435bbec1ba83/a2b9d01a-f05c-4fe0-bfaf-c74e95793a8f"
-					(reference "C29")
+					(reference "C1105")
 					(unit 1)
 				)
@@
 		(in_pos_files yes)
 		(dnp no)
-		(property "Reference" "C56"
+		(property "Reference" "C1103"
 			(at 182.372 82.3022 0)
 			(show_name no)
@@
 			)
 		)
-		(property "Value" "0.01uF"
+		(property "Value" "10nF"
 			(at 182.372 84.074 0)
 			(show_name no)
@@
 			(project "gridfins"
 				(path "/7db990e4-92e1-4f99-b4d2-435bbec1ba83/a2b9d01a-f05c-4fe0-bfaf-c74e95793a8f"
-					(reference "C56")
+					(reference "C1103")
 					(unit 1)
 				)
@@
 		(dnp no)
 		(fields_autoplaced yes)
-		(property "Reference" "R46"
+		(property "Reference" "R1104"
 			(at 82.55 62.2299 0)
 			(show_name no)
@@
 			)
 		)
-		(property "Value" "10k"
+		(property "Value" "10kΩ"
 			(at 82.55 64.7699 0)
 			(show_name no)
@@
 			(project "gridfins"
 				(path "/7db990e4-92e1-4f99-b4d2-435bbec1ba83/a2b9d01a-f05c-4fe0-bfaf-c74e95793a8f"
-					(reference "R46")
+					(reference "R1104")
 					(unit 1)
 				)
@@
 		(in_pos_files yes)
 		(dnp no)
-		(property "Reference" "#PWR0118"
+		(property "Reference" "#PWR01106"
 			(at 187.96 99.06 0)
 			(hide yes)
@@
 			(project "gridfins"
 				(path "/7db990e4-92e1-4f99-b4d2-435bbec1ba83/a2b9d01a-f05c-4fe0-bfaf-c74e95793a8f"
-					(reference "#PWR0118")
+					(reference "#PWR01106")
 					(unit 1)
 				)
@@
 		(in_pos_files yes)
 		(dnp no)
-		(property "Reference" "C30"
+		(property "Reference" "C1106"
 			(at 210.312 76.454 0)
 			(show_name no)
@@
 			(project "gridfins"
 				(path "/7db990e4-92e1-4f99-b4d2-435bbec1ba83/a2b9d01a-f05c-4fe0-bfaf-c74e95793a8f"
-					(reference "C30")
+					(reference "C1106")
 					(unit 1)
 				)
@@
 		(in_pos_files yes)
 		(dnp no)
-		(property "Reference" "C57"
+		(property "Reference" "C1101"
 			(at 182.6198 71.628 0)
 			(hide yes)
@@
 			(project "gridfins"
 				(path "/7db990e4-92e1-4f99-b4d2-435bbec1ba83/a2b9d01a-f05c-4fe0-bfaf-c74e95793a8f"
-					(reference "C57")
+					(reference "C1101")
 					(unit 1)
 				)
@@
 		(in_pos_files yes)
 		(dnp no)
-		(property "Reference" "#PWR090"
+		(property "Reference" "#PWR01104"
 			(at 175.26 76.2 0)
 			(hide yes)
@@
 			(project "gridfins"
 				(path "/7db990e4-92e1-4f99-b4d2-435bbec1ba83/a2b9d01a-f05c-4fe0-bfaf-c74e95793a8f"
-					(reference "#PWR090")
+					(reference "#PWR01104")
 					(unit 1)
 				)
@@
 		(in_pos_files yes)
 		(dnp no)
-		(property "Reference" "C19"
+		(property "Reference" "C1102"
 			(at 182.8136 76.708 0)
 			(show_name no)
@@
 			)
 		)
-		(property "Value" "0.01uF"
+		(property "Value" "10nF"
 			(at 181.7976 78.486 0)
 			(show_name no)
@@
 			(project "gridfins"
 				(path "/7db990e4-92e1-4f99-b4d2-435bbec1ba83/a2b9d01a-f05c-4fe0-bfaf-c74e95793a8f"
-					(reference "C19")
+					(reference "C1102")
 					(unit 1)
 				)
@@
 		(in_pos_files yes)
 		(dnp no)
-		(property "Reference" "#PWR028"
+		(property "Reference" "#PWR01108"
 			(at 223.52 81.28 0)
 			(hide yes)
@@
 			(project "gridfins"
 				(path "/7db990e4-92e1-4f99-b4d2-435bbec1ba83/a2b9d01a-f05c-4fe0-bfaf-c74e95793a8f"
-					(reference "#PWR028")
+					(reference "#PWR01108")
 					(unit 1)
 				)
@@
 		(in_pos_files yes)
 		(dnp no)
-		(property "Reference" "R44"
+		(property "Reference" "R1106"
 			(at 177.546 96.774 90)
 			(show_name no)
@@
 			)
 		)
-		(property "Value" "0.5"
+		(property "Value" "0.5Ω"
 			(at 177.8 98.552 90)
 			(show_name no)
@@
 			(project "gridfins"
 				(path "/7db990e4-92e1-4f99-b4d2-435bbec1ba83/a2b9d01a-f05c-4fe0-bfaf-c74e95793a8f"
-					(reference "R44")
-					(unit 1)
-				)
+					(reference "R1106")
+					(unit 1)
+				)
