File: gridfins/SD_sch.kicad_sch (KiCad schematic)
At the start: 6 parts, among them J6 ST1W008S4TR2000, Q3 DMP3099

Commit message: formatting
Parts:
- C801: renamed from C51; value 0.1uF -> 100nF
- JP801: renamed from JP34; now left out of the parts list
- R801: renamed from R71; value 1k -> 1kΩ
- R802: renamed from R30; value 10k -> 10kΩ
- renumbered J6 to J801, Q3 to Q801
Other:
- moved on the sheet: JP801
Changed lines of the file:
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@@
 	(wire
 		(pts
-			(xy 115.57 88.138) (xy 115.57 87.122)
+			(xy 111.76 88.138) (xy 111.76 86.36)
 		)
 		(stroke
@@
 	(wire
 		(pts
-			(xy 115.57 77.47) (xy 128.016 77.47)
+			(xy 111.76 77.47) (xy 128.016 77.47)
 		)
 		(stroke
@@
 	(wire
 		(pts
-			(xy 128.016 88.138) (xy 115.57 88.138)
+			(xy 128.016 88.138) (xy 111.76 88.138)
 		)
 		(stroke
@@
 	(wire
 		(pts
-			(xy 115.57 79.502) (xy 115.57 77.47)
+			(xy 111.76 78.74) (xy 111.76 77.47)
 		)
 		(stroke
@@
 	(symbol
 		(lib_id "Jumper:SolderJumper_2_Open")
-		(at 115.57 83.312 270)
+		(at 111.76 82.55 270)
 		(unit 1)
 		(body_style 1)
 		(exclude_from_sim no)
-		(in_bom yes)
+		(in_bom no)
 		(on_board yes)
 		(in_pos_files yes)
 		(dnp no)
-		(property "Reference" "JP34"
-			(at 110.49 83.312 0)
+		(property "Reference" "JP801"
+			(at 106.68 82.55 90)
 			(show_name no)
 			(do_not_autoplace no)
@@
 		)
 		(property "Value" "SolderJumper_2_Open"
-			(at 83.82 65.532 0)
+			(at 80.01 64.77 0)
 			(hide yes)
 			(show_name no)
@@
 		)
 		(property "Footprint" "iclr:SmallerSolderJP"
-			(at 115.57 83.312 0)
+			(at 111.76 82.55 0)
 			(hide yes)
 			(show_name no)
@@
 		)
 		(property "Datasheet" ""
-			(at 115.57 83.312 0)
+			(at 111.76 82.55 0)
 			(hide yes)
 			(show_name no)
@@
 		)
 		(property "Description" ""
-			(at 115.57 83.312 0)
+			(at 111.76 82.55 0)
 			(hide yes)
 			(show_name no)
@@
 			(project "gridfins"
 				(path "/7db990e4-92e1-4f99-b4d2-435bbec1ba83/5e350498-f93c-4da7-ae1f-748ce4c04899"
-					(reference "JP34")
+					(reference "JP801")
 					(unit 1)
 				)
@@
 		(in_pos_files yes)
 		(dnp no)
-		(property "Reference" "#PWR089"
+		(property "Reference" "#PWR0805"
 			(at 148.844 76.962 0)
 			(hide yes)
@@
 			(project "gridfins"
 				(path "/7db990e4-92e1-4f99-b4d2-435bbec1ba83/5e350498-f93c-4da7-ae1f-748ce4c04899"
-					(reference "#PWR089")
+					(reference "#PWR0805")
 					(unit 1)
 				)
@@
 		(in_pos_files yes)
 		(dnp no)
-		(property "Reference" "R71"
-			(at 132.969 85.7281 0)
-			(show_name no)
-			(do_not_autoplace no)
-			(effects
-				(font
-					(size 1.27 1.27)
-				)
-			)
-		)
-		(property "Value" "1k"
-			(at 132.969 88.265 0)
+		(property "Reference" "R801"
+			(at 140.462 84.836 0)
+			(show_name no)
+			(do_not_autoplace no)
+			(effects
+				(font
+					(size 1.27 1.27)
+				)
+			)
+		)
+		(property "Value" "1kΩ"
+			(at 140.462 87.3729 0)
 			(show_name no)
 			(do_not_autoplace no)
@@
 			(project "gridfins"
 				(path "/7db990e4-92e1-4f99-b4d2-435bbec1ba83/5e350498-f93c-4da7-ae1f-748ce4c04899"
-					(reference "R71")
+					(reference "R801")
 					(unit 1)
 				)
@@
 		(in_pos_files yes)
 		(dnp no)
-		(property "Reference" "#PWR088"
+		(property "Reference" "#PWR0803"
 			(at 129.032 108.458 0)
 			(hide yes)
@@
 			(project "gridfins"
 				(path "/7db990e4-92e1-4f99-b4d2-435bbec1ba83/5e350498-f93c-4da7-ae1f-748ce4c04899"
-					(reference "#PWR088")
+					(reference "#PWR0803")
 					(unit 1)
 				)
@@
 		(dnp no)
 		(fields_autoplaced yes)
-		(property "Reference" "Q3"
+		(property "Reference" "Q801"
 			(at 124.206 81.788 0)
 			(show_name no)
@@
 			(project "gridfins"
 				(path "/7db990e4-92e1-4f99-b4d2-435bbec1ba83/5e350498-f93c-4da7-ae1f-748ce4c04899"
-					(reference "Q3")
+					(reference "Q801")
 					(unit 1)
 				)
@@
 		(dnp no)
 		(fields_autoplaced yes)
-		(property "Reference" "#PWR095"
+		(property "Reference" "#PWR0802"
 			(at 128.016 80.264 0)
 			(hide yes)
@@
 			(project "gridfins"
 				(path "/7db990e4-92e1-4f99-b4d2-435bbec1ba83/5e350498-f93c-4da7-ae1f-748ce4c04899"
-					(reference "#PWR095")
+					(reference "#PWR0802")
 					(unit 1)
 				)
@@
 		(in_pos_files yes)
 		(dnp no)
-		(property "Reference" "R30"
+		(property "Reference" "R802"
 			(at 145.034 73.152 0)
 			(show_name no)
@@
 			)
 		)
-		(property "Value" "10k"
+		(property "Value" "10kΩ"
 			(at 145.034 75.692 0)
 			(show_name no)
@@
 			(project "gridfins"
 				(path "/7db990e4-92e1-4f99-b4d2-435bbec1ba83/5e350498-f93c-4da7-ae1f-748ce4c04899"
-					(reference "R30")
+					(reference "R802")
 					(unit 1)
 				)
@@
 		(in_pos_files yes)
 		(dnp no)
-		(property "Reference" "C51"
+		(property "Reference" "C801"
 			(at 119.126 91.948 0)
 			(show_name no)
@@
 			)
 		)
-		(property "Value" "0.1uF"
+		(property "Value" "100nF"
 			(at 119.126 94.2594 0)
 			(show_name no)
@@
 			(project "gridfins"
 				(path "/7db990e4-92e1-4f99-b4d2-435bbec1ba83/5e350498-f93c-4da7-ae1f-748ce4c04899"
-					(reference "C51")
+					(reference "C801")
 					(unit 1)
 				)
@@
 		(dnp no)
 		(fields_autoplaced yes)
-		(property "Reference" "J6"
+		(property "Reference" "J801"
 			(at 162.814 77.6435 0)
 			(show_name no)
@@
 			(project "gridfins"
 				(path "/7db990e4-92e1-4f99-b4d2-435bbec1ba83/5e350498-f93c-4da7-ae1f-748ce4c04899"
-					(reference "J6")
+					(reference "J801")
 					(unit 1)
 				)
@@
 		(in_pos_files yes)
 		(dnp no)
-		(property "Reference" "#PWR094"
+		(property "Reference" "#PWR0801"
 			(at 124.206 100.838 0)
 			(hide yes)
@@
 			(project "gridfins"
 				(path "/7db990e4-92e1-4f99-b4d2-435bbec1ba83/5e350498-f93c-4da7-ae1f-748ce4c04899"
-					(reference "#PWR094")
+					(reference "#PWR0801")
 					(unit 1)
 				)
@@
 		(dnp no)
 		(fields_autoplaced yes)
-		(property "Reference" "#PWR0154"
+		(property "Reference" "#PWR0804"
 			(at 136.398 94.488 0)
 			(hide yes)
@@
 			(project "gridfins"
 				(path "/7db990e4-92e1-4f99-b4d2-435bbec1ba83/5e350498-f93c-4da7-ae1f-748ce4c04899"
-					(reference "#PWR0154")
+					(reference "#PWR0804")
 					(unit 1)
 				)
@@
 		(dnp no)
 		(fields_autoplaced yes)
-		(property "Reference" "#PWR0157"
+		(property "Reference" "#PWR0806"
 			(at 178.054 121.158 0)
 			(hide yes)
@@
 			(project "gridfins"
 				(path "/7db990e4-92e1-4f99-b4d2-435bbec1ba83/5e350498-f93c-4da7-ae1f-748ce4c04899"
-					(reference "#PWR0157")
+					(reference "#PWR0806")
 					(unit 1)
 				)
