File: gridfins/actuators.kicad_sch (KiCad schematic)
At the start: 10 parts, among them J3 ServoCH0, J4 ServoCH1, J5 ServoCH2

Commit message: feat: Massive changes, board almost ready for review
Parts:
- removed D4, D5, D6, D7: ~, Package_TO_SOT_SMD:SOT-353_SC-70-5, symbol iclr:CPDV5-3V3UP
- added D3, D4, D5: CPDF3V3UP-HF, iclr:CPD, symbol iclr:CPDF3V3UP-HF
Connections:
- net GND: now also D3.1, D4.1, D5.1
- net Servo_0_PWM: now also D3.2
- net Servo_1_PWM: now also D4.2
- net Servo_2_PWM: now also D5.2
- no-connect marks 1 -> 0

Commit message: formatting
Parts:
- R1001: renamed from R25; value 165R -> 165Ω
- R1002: renamed from R26; value 165R -> 165Ω
- R1003: renamed from R27; value 165R -> 165Ω
- renumbered D3 to D1001, D5 to D1002, D4 to D1003, J3 to J1001, J4 to J1002, J5 to J1003
Changed lines of the file:
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@@
 		(dnp no)
 		(fields_autoplaced yes)
-		(property "Reference" "#PWR0110"
+		(property "Reference" "#PWR01002"
 			(at 93.98 140.97 0)
 			(hide yes)
@@
 			(project "gridfins"
 				(path "/7db990e4-92e1-4f99-b4d2-435bbec1ba83/4a649bbd-9e5c-4376-be49-6107979e6dfc"
-					(reference "#PWR0110")
+					(reference "#PWR01002")
 					(unit 1)
 				)
@@
 		(dnp no)
 		(fields_autoplaced yes)
-		(property "Reference" "R26"
+		(property "Reference" "R1002"
 			(at 144.78 96.52 90)
 			(show_name no)
@@
 			)
 		)
-		(property "Value" "165R"
+		(property "Value" "165Ω"
 			(at 144.78 99.06 90)
 			(show_name no)
@@
 			(project "gridfins"
 				(path "/7db990e4-92e1-4f99-b4d2-435bbec1ba83/4a649bbd-9e5c-4376-be49-6107979e6dfc"
-					(reference "R26")
+					(reference "R1002")
 					(unit 1)
 				)
@@
 		(dnp no)
 		(fields_autoplaced yes)
-		(property "Reference" "D3"
+		(property "Reference" "D1001"
 			(at 91.44 87.5791 90)
 			(show_name no)
@@
 			(project "gridfins"
 				(path "/7db990e4-92e1-4f99-b4d2-435bbec1ba83/4a649bbd-9e5c-4376-be49-6107979e6dfc"
-					(reference "D3")
+					(reference "D1001")
 					(unit 1)
 				)
@@
 		(dnp no)
 		(fields_autoplaced yes)
-		(property "Reference" "#PWR0101"
+		(property "Reference" "#PWR01003"
 			(at 101.6 99.06 0)
 			(hide yes)
@@
 			(project "gridfins"
 				(path "/7db990e4-92e1-4f99-b4d2-435bbec1ba83/4a649bbd-9e5c-4376-be49-6107979e6dfc"
-					(reference "#PWR0101")
+					(reference "#PWR01003")
 					(unit 1)
 				)
@@
 		(dnp no)
 		(fields_autoplaced yes)
-		(property "Reference" "#PWR0104"
+		(property "Reference" "#PWR01004"
 			(at 135.89 92.71 0)
 			(hide yes)
@@
 			(project "gridfins"
 				(path "/7db990e4-92e1-4f99-b4d2-435bbec1ba83/4a649bbd-9e5c-4376-be49-6107979e6dfc"
-					(reference "#PWR0104")
+					(reference "#PWR01004")
 					(unit 1)
 				)
@@
 		(dnp no)
 		(fields_autoplaced yes)
-		(property "Reference" "J5"
+		(property "Reference" "J1003"
 			(at 156.21 119.3799 0)
 			(show_name no)
@@
 			(project "gridfins"
 				(path "/7db990e4-92e1-4f99-b4d2-435bbec1ba83/4a649bbd-9e5c-4376-be49-6107979e6dfc"
-					(reference "J5")
+					(reference "J1003")
 					(unit 1)
 				)
@@
 		(dnp no)
 		(fields_autoplaced yes)
-		(property "Reference" "#PWR0106"
+		(property "Reference" "#PWR01006"
 			(at 138.43 124.46 0)
 			(hide yes)
@@
 			(project "gridfins"
 				(path "/7db990e4-92e1-4f99-b4d2-435bbec1ba83/4a649bbd-9e5c-4376-be49-6107979e6dfc"
-					(reference "#PWR0106")
+					(reference "#PWR01006")
 					(unit 1)
 				)
@@
 		(dnp no)
 		(fields_autoplaced yes)
-		(property "Reference" "#PWR0108"
+		(property "Reference" "#PWR01008"
 			(at 143.51 106.68 0)
 			(hide yes)
@@
 			(project "gridfins"
 				(path "/7db990e4-92e1-4f99-b4d2-435bbec1ba83/4a649bbd-9e5c-4376-be49-6107979e6dfc"
-					(reference "#PWR0108")
+					(reference "#PWR01008")
 					(unit 1)
 				)
@@
 		(dnp no)
 		(fields_autoplaced yes)
-		(property "Reference" "#PWR0107"
+		(property "Reference" "#PWR01007"
 			(at 143.51 91.44 0)
 			(hide yes)
@@
 			(project "gridfins"
 				(path "/7db990e4-92e1-4f99-b4d2-435bbec1ba83/4a649bbd-9e5c-4376-be49-6107979e6dfc"
-					(reference "#PWR0107")
+					(reference "#PWR01007")
 					(unit 1)
 				)
@@
 		(dnp no)
 		(fields_autoplaced yes)
-		(property "Reference" "D5"
+		(property "Reference" "D1002"
 			(at 96.52 128.2191 90)
 			(show_name no)
@@
 			(project "gridfins"
 				(path "/7db990e4-92e1-4f99-b4d2-435bbec1ba83/4a649bbd-9e5c-4376-be49-6107979e6dfc"
-					(reference "D5")
+					(reference "D1002")
 					(unit 1)
 				)
@@
 		(dnp no)
 		(fields_autoplaced yes)
-		(property "Reference" "J3"
+		(property "Reference" "J1001"
 			(at 156.21 87.6299 0)
 			(show_name no)
@@
 			(project "gridfins"
 				(path "/7db990e4-92e1-4f99-b4d2-435bbec1ba83/4a649bbd-9e5c-4376-be49-6107979e6dfc"
-					(reference "J3")
+					(reference "J1001")
 					(unit 1)
 				)
@@
 		(dnp no)
 		(fields_autoplaced yes)
-		(property "Reference" "J4"
+		(property "Reference" "J1002"
 			(at 156.21 102.8699 0)
 			(show_name no)
@@
 			(project "gridfins"
 				(path "/7db990e4-92e1-4f99-b4d2-435bbec1ba83/4a649bbd-9e5c-4376-be49-6107979e6dfc"
-					(reference "J4")
+					(reference "J1002")
 					(unit 1)
 				)
@@
 		(dnp no)
 		(fields_autoplaced yes)
-		(property "Reference" "R27"
+		(property "Reference" "R1003"
 			(at 144.78 113.03 90)
 			(show_name no)
@@
 			)
 		)
-		(property "Value" "165R"
+		(property "Value" "165Ω"
 			(at 144.78 115.57 90)
 			(show_name no)
@@
 			(project "gridfins"
 				(path "/7db990e4-92e1-4f99-b4d2-435bbec1ba83/4a649bbd-9e5c-4376-be49-6107979e6dfc"
-					(reference "R27")
+					(reference "R1003")
 					(unit 1)
 				)
@@
 		(dnp no)
 		(fields_autoplaced yes)
-		(property "Reference" "#PWR0103"
+		(property "Reference" "#PWR01009"
 			(at 143.51 123.19 0)
 			(hide yes)
@@
 			(project "gridfins"
 				(path "/7db990e4-92e1-4f99-b4d2-435bbec1ba83/4a649bbd-9e5c-4376-be49-6107979e6dfc"
-					(reference "#PWR0103")
+					(reference "#PWR01009")
 					(unit 1)
 				)
@@
 		(dnp no)
 		(fields_autoplaced yes)
-		(property "Reference" "R25"
+		(property "Reference" "R1001"
 			(at 144.78 81.28 90)
 			(show_name no)
@@
 			)
 		)
-		(property "Value" "165R"
+		(property "Value" "165Ω"
 			(at 144.78 83.82 90)
 			(show_name no)
@@
 			(project "gridfins"
 				(path "/7db990e4-92e1-4f99-b4d2-435bbec1ba83/4a649bbd-9e5c-4376-be49-6107979e6dfc"
-					(reference "R25")
+					(reference "R1001")
 					(unit 1)
 				)
@@
 		(dnp no)
 		(fields_autoplaced yes)
-		(property "Reference" "#PWR0102"
+		(property "Reference" "#PWR01001"
 			(at 93.98 99.06 0)
 			(hide yes)
@@
 			(project "gridfins"
 				(path "/7db990e4-92e1-4f99-b4d2-435bbec1ba83/4a649bbd-9e5c-4376-be49-6107979e6dfc"
-					(reference "#PWR0102")
+					(reference "#PWR01001")
 					(unit 1)
 				)
@@
 		(dnp no)
 		(fields_autoplaced yes)
-		(property "Reference" "D4"
+		(property "Reference" "D1003"
 			(at 104.14 87.5791 90)
 			(show_name no)
@@
 			(project "gridfins"
 				(path "/7db990e4-92e1-4f99-b4d2-435bbec1ba83/4a649bbd-9e5c-4376-be49-6107979e6dfc"
-					(reference "D4")
+					(reference "D1003")
 					(unit 1)
 				)
@@
 		(dnp no)
 		(fields_autoplaced yes)
-		(property "Reference" "#PWR0105"
+		(property "Reference" "#PWR01005"
 			(at 138.43 107.95 0)
 			(hide yes)
@@
 			(project "gridfins"
 				(path "/7db990e4-92e1-4f99-b4d2-435bbec1ba83/4a649bbd-9e5c-4376-be49-6107979e6dfc"
-					(reference "#PWR0105")
-					(unit 1)
-				)
+					(reference "#PWR01005")
+					(unit 1)
+				)
