File: gridfins/highside.kicad_sch (KiCad schematic)
At the start: 11 parts, among them Q5 BSZ025N04LS, Q6 BSZ025N04LS, U10 LM74810

Commit message: formatting
Parts:
- C301: renamed from C52; value 0.1uF -> 100nF
- C303: renamed from C54; value 0.1uF -> 100nF
- C304: renamed from C55; value 0.1uF -> 100nF
- R301: renamed from R31; value 10k -> 10kΩ
- R302: renamed from R32; value 100k -> 100kΩ
- R303: renamed from R33; value 5.1k -> 5.1kΩ
- R304: renamed from R35; value 4.22k -> 4.22kΩ
- renumbered C53 to C302, Q5 to Q301, Q6 to Q302, U10 to U301
Other:
- moved on the sheet: R302, R303, R304
