File: gridfins/power.kicad_sch (KiCad schematic)
At the start: 20 parts, among them U3 LM66200DRLR, U4 MAX77827AEFD+T, U5 SC4215ASTRT

Commit message: formatting
Parts:
- C208: renamed from C27; value 0.1uF -> 100nF
- R201: renamed from R14; value 10k -> 10kΩ
- R202: renamed from R15; value 14k -> 14kΩ
- R203: renamed from R16; value 56k -> 56kΩ
- R204: renamed from R17; value 10k -> 10kΩ
- TP201: renamed from TP4; now left out of the parts list
- TP202: renamed from TP5; now left out of the parts list
- TP203: renamed from TP6; now left out of the parts list
- TP204: renamed from TP8; now left out of the parts list
- renumbered C20 to C201, C21 to C202, C22 to C203, C23 to C204, C24 to C205, C25 to C206, C26 to C207, L3 to L201, U3 to U201, U4 to U202, U5 to U203
