File: gridfins/usb.kicad_sch (KiCad schematic)
At the start: 8 parts, among them J2 USB_C_Receptacle_USB2.0

Commit message: formatting
Parts:
- LED601: renamed from LED6; value WHITE_LED -> LED_WHITE
- R601: renamed from R11; value 5.1k -> 5.1kΩ
- R602: renamed from R12; value 5.1k -> 5.1kΩ
- R603: renamed from R13; value 5.1k -> 5.1kΩ
- TP601: renamed from TP1; now left out of the parts list
- TP602: renamed from TP2; now left out of the parts list
- renumbered D2 to D601, J2 to J601
Other:
- moved on the sheet: R601, R602
