File: gridfins/buck_SERVO.kicad_sch (KiCad schematic)
At the start: 30 parts, among them Q4 SSM3K15AMFV,L3F, U12 SiC437AED-T1

Commit message: formatting
Parts:
- removed C80: 1uF, Capacitor_SMD:C_0402_1005Metric, symbol Device:C_Small
- removed C81: 4.7uF, Capacitor_SMD:C_0402_1005Metric, symbol Device:C_Small
- removed C82, C92: 100uF, Capacitor_Tantalum_SMD:CP_EIA-7360-38_Kemet-E, symbol Device:C_Polarized_Small
- removed C83, C84, C86, C87, C88, C91, C93, C94, C95, C96: 47uF, Capacitor_SMD:C_1206_3216Metric, symbol Device:C_Small
- removed C85: 100nF, Capacitor_SMD:C_0402_1005Metric, symbol Device:C_Small
- removed C89: 0.1uF, Capacitor_SMD:C_0402_1005Metric, symbol Device:C_Small
- removed C90: 160pF, Capacitor_SMD:C_0603_1608Metric, symbol Device:C_Small
- removed L6: 3.3uH, iclr:IND_SPM10065VT-3R3M-D, symbol Device:L
- removed Q4: SSM3K15AMFV,L3F, iclr:SOT-723, symbol Device:Q_NMOS_GSD
- removed R58, R60, R66: 10k, Resistor_SMD:R_0402_1005Metric, symbol Device:R_Small
- removed R59: 113k, Resistor_SMD:R_0402_1005Metric, symbol Device:R_Small
- removed R61: 2.2, Resistor_SMD:R_0402_1005Metric, symbol Device:R_Small
- removed R62: 1k, Resistor_SMD:R_0402_1005Metric, symbol Device:R_Small
- removed R63: 442k, Resistor_SMD:R_0402_1005Metric, symbol Device:R_Small
- removed R64: 200k, Resistor_SMD:R_0402_1005Metric, symbol Device:R_Small
- removed R65: 100k, Resistor_SMD:R_0402_1005Metric, symbol Device:R_Small
- removed R67: 5.1R, Resistor_SMD:R_0603_1608Metric, symbol Device:R_Small
- removed U12: SiC437AED-T1, iclr:SiC437BEDT1GE3, symbol iclr:SiC437BED-T1-GE3
- added C401: 1uF, Capacitor_SMD:C_0402_1005Metric, symbol Device:C_Small
- added C402: 4.7uF, Capacitor_SMD:C_0402_1005Metric, symbol Device:C_Small
- added C403, C413: 100uF, Capacitor_Tantalum_SMD:CP_EIA-7360-38_Kemet-E, symbol Device:C_Polarized_Small
- added C404, C405, C407, C408, C409, C412, C414, C415, C416, C417: 47uF, Capacitor_SMD:C_1206_3216Metric, symbol Device:C_Small
- added C406, C410: 100nF, Capacitor_SMD:C_0402_1005Metric, symbol Device:C_Small
- added C411: 160pF, Capacitor_SMD:C_0603_1608Metric, symbol Device:C_Small
- added L401: 3.3uH, iclr:IND_SPM10065VT-3R3M-D, symbol Device:L
- added Q401: SSM3K15AMFV,L3F, iclr:SOT-723, symbol Device:Q_NMOS_GSD
- added R401, R403, R409: 10kΩ, Resistor_SMD:R_0402_1005Metric, symbol Device:R_Small
- added R402: 113kΩ, Resistor_SMD:R_0402_1005Metric, symbol Device:R_Small
- added R404: 2.2Ω, Resistor_SMD:R_0402_1005Metric, symbol Device:R_Small
- added R405: 1kΩ, Resistor_SMD:R_0402_1005Metric, symbol Device:R_Small
- added R406: 442kΩ, Resistor_SMD:R_0402_1005Metric, symbol Device:R_Small
- added R407: 200kΩ, Resistor_SMD:R_0402_1005Metric, symbol Device:R_Small
- added R408: 100kΩ, Resistor_SMD:R_0402_1005Metric, symbol Device:R_Small
- added R410: 5.1Ω, Resistor_SMD:R_0603_1608Metric, symbol Device:R_Small
- added U401: SiC437AED-T1, iclr:SiC437BEDT1GE3, symbol iclr:SiC437BED-T1-GE3
Connections:
- net +7.4V: now also C404.1, C405.1, C407.1, C408.1, C409.1, C412.2, C414.1, C415.1, C416.1, C417.1, L401.1, R402.2, R406.2, U401.18 (V_OUT)
- net BOOT: now also C410.1, U401.23 (BOOT)
- net BUCK_EN: now also Q401.1 (G), R405.2
- net EN: now also Q401.3 (D), R409.1, U401.19 (EN)
- net FB: now also R402.1, R403.2, R406.1, U401.17 (FB)
- net GND: now also C401.1, C402.1, C403.2, C404.2, C405.2, C406.2, C407.2, C408.2, C409.2, C412.1, C413.2, C414.2, C415.2, C416.2, C417.2, Q401.2 (S), R403.1, R405.1, R408.2, R410.2, U401.13 (P_GND_3), U401.16 (A_GND), U401.25 (AGND), U401.27 (PGND), U401.29 (P_GND_4), U401.3 (P_GND_1), U401.4 (P_GND_2)
- net PGOOD: now also R401.2, U401.14 (P_GOOD)
- net PHASE: now also R404.1, U401.24 (PHASE)
- net SW: now also C411.1, L401.2, U401.30 (SW_6), U401.5 (SW_1), U401.6 (SW_2), U401.7 (SW_3), U401.8 (SW_4), U401.9 (SW_5)
- net VDD: now also C401.2, R401.1, R407.2, U401.15 (VDD)
- net VINBuck: now also C403.1, C406.1, C413.1, R409.2, U401.1 (V_IN_1), U401.2 (V_IN_2), U401.22 (VIN_1), U401.26 (VIN_2)
- new net: C411.2, R410.1
- new net: C402.2, U401.12 (V_DRV)
- new net: R407.1, U401.20 (MODE_2)
- new net: R408.1, U401.21 (_MODE_1)
- new net: C410.2, R404.2
Other:
- note removed: "SPM10065VT-3R3M-D"

Commit message: feat: Post Jack review
Changed buck inductors to be wuerth. Reduced board footprint. Incorporated review feedback
Parts:
- L401: footprint iclr:IND_SPM10065VT-3R3M-D -> iclr:WE-XHMI_7070
Connections:
- net +7.4V: now also L401.2; no longer L401.1
- net SW: now also L401.1; no longer L401.2
Other:
- moved on the sheet: L401
Changed lines of the file:
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@@
 	(symbol
 		(lib_id "Device:L")
-		(at 59.69 81.28 90)
+		(at 59.69 81.28 270)
+		(mirror x)
 		(unit 1)
 		(body_style 1)
@@
 			)
 		)
-		(property "Footprint" "iclr:IND_SPM10065VT-3R3M-D"
+		(property "Footprint" "iclr:WE-XHMI_7070"
 			(at 59.69 81.28 0)
 			(hide yes)
