File: gridfins/gridfins.kicad_sch (KiCad schematic)
At the start: 49 parts, among them J1 RBUS, U1 ESP32-S3, Y1 R940000171

Commit message: feat: Massive changes, board almost ready for review
Parts:
- removed J1: RBUS, iclr:Molex_Mini-Fit_Jr_5569-06A2_2x03_P4.20mm_Horizontal, symbol Connector:Conn_01x06_Male
- removed JP2, JP3: Conn_01x02_Male, Connector_PinHeader_2.54mm:PinHeader_1x02_P2.54mm_Vertical, symbol Connector:Conn_01x02_Male
- removed TP3: TestPoint, TestPoint:TestPoint_Pad_D1.0mm, symbol Connector:TestPoint
- added J1: RBUS, iclr:Molex_Mini-Fit_Jr_5569-08A2_2x04_P4.20mm_Horizontal, symbol Connector:Conn_01x08_Pin
- added J10: Limit switch 2, Connector_PinHeader_2.54mm:PinHeader_1x02_P2.54mm_Vertical, symbol Connector:Conn_01x02_Pin
- added J11: Conn_01x03_Pin, Connector_PinHeader_1.00mm:PinHeader_1x03_P1.00mm_Vertical, symbol Connector:Conn_01x03_Pin
- added J7: Encoder breakout, Connector_PinHeader_2.54mm:PinHeader_2x03_P2.54mm_Vertical, symbol Connector:Conn_01x06_Pin
- added J9: Limit switch 1, Connector_PinHeader_2.54mm:PinHeader_1x02_P2.54mm_Vertical, symbol Connector:Conn_01x02_Pin
- added R48, R49: 10k, Resistor_SMD:R_0402_1005Metric, symbol Device:R
- added TP11, TP13, TP14: TestPoint, TestPoint:TestPoint_Pad_D1.0mm, symbol Connector:TestPoint
Connections:
- net +12V is gone; now on net +10V: R7.1
- net BUCK_EN is gone; now on net MAG_CS: U1.51 (GPIO45)
- net +3V3: now also J7.1 (Pin_1), R48.2, R49.2
- net BOOT: now also J11.3 (Pin_3)
- net BUS_VMON: now also U1.24 (GPIO18/ADC2_CH7/DAC_1); no longer U1.6 (GPIO1/ADC1_CH0)
- net CAN+: now also J1.7 (Pin_7)
- net CAN-: now also J1.8 (Pin_8)
- net CAN_RX: now also U1.15 (GPIO10/ADC1_CH9)
- net CAN_TX: now also U1.16 (GPIO11/ADC2_CH0)
- net CHIP_PU: now also C3.2, J11.1 (Pin_1); no longer C3.1
- net DIR/BPHASE: now also U1.39 (GPIO34); no longer U1.24 (GPIO18/ADC2_CH7/DAC_1)
- net ENCODER_CS: now also U1.14 (GPIO9/ADC1_CH8), J7.3 (Pin_3); no longer U1.43 (GPIO38)
- net GND: now also C3.1, J1.1 (Pin_1), J1.2 (Pin_2), J1.3 (Pin_3), J10.2 (Pin_2), J11.2 (Pin_2), J7.2 (Pin_2), J9.2 (Pin_2); no longer C3.2
- net HSIDE_EN: now also U1.17 (GPIO12/ADC2_CH1); no longer U1.42 (GPIO37)
- net HSPI_MISO: now also U1.44 (MTCK/JTAG/GPIO39); no longer U1.14 (GPIO9/ADC1_CH8)
- net HSPI_MOSI: now also U1.42 (GPIO37); no longer U1.15 (GPIO10/ADC1_CH9)
- net HSPI_SCLK: now also U1.43 (GPIO38); no longer U1.16 (GPIO11/ADC2_CH0)
- net IMU1_CS: now also U1.47 (MTDI/JTAG/GPIO41); no longer U1.17 (GPIO12/ADC2_CH1)
- net IMU2_CS: now also U1.48 (MTMS/JTAG/GPIO42); no longer U1.18 (GPIO13/ADC2_CH2)
- net M0/APHASE: now also U1.27 (GPIO21); no longer U1.23 (GPIO17/ADC2_CH6/DAC_2)
- net MAG_CS: no longer U1.19 (GPIO14/ADC2_CH3)
- net NENBL/AENBL: now also U1.41 (GPIO36); no longer U1.27 (GPIO21)
- net NSLEEP: now also U1.38 (GPIO33); no longer U1.22 (GPIO16/ADC2_CH5/XTAL_32K_N)
- net RBUS_uC_V: now also J1.4 (Pin_4)
- net SD1_CS: now also U1.13 (GPIO8/ADC1_CH7); no longer U1.10 (GPIO5/ADC1_CH4)
- net SERVOPWM0: now also U1.23 (GPIO17/ADC2_CH6/DAC_2); no longer U1.39 (GPIO34)
- net SERVOPWM1: now also U1.22 (GPIO16/ADC2_CH5/XTAL_32K_N); no longer U1.40 (GPIO35)
- net SERVOPWM2: now also U1.21 (GPIO15/ADC2_CH4/XTAL_32K_P); no longer U1.41 (GPIO36)
- net STEP/BENBL: now also U1.40 (GPIO35); no longer U1.21 (GPIO15/ADC2_CH4/XTAL_32K_P)
- net ServoV_LOG: now also TP14.1
- net VSPI_MISO: now also U1.10 (GPIO5/ADC1_CH4), J7.6 (Pin_6); no longer U1.13 (GPIO8/ADC1_CH7)
- net VSPI_MOSI: now also J7.4 (Pin_4)
- net VSPI_SCLK: now also J7.5 (Pin_5)
- net M1: now reaches U1.36 (SPICLK_N/GPIO48)
- net Fault: now reaches U1.37 (SPICLK_P/GPIO47)
- net Switch_1: now reaches U1.45 (MTDO/JTAG/GPIO40)
- net Switch_1: now also J10.1 (Pin_1), R49.1
- net BuckPGOOD renamed BuckPGOOD_H
- net BuckPGOOD_H: now also TP11.1; no longer R45.2
- new net BUCK_EN_H: U1.18 (GPIO13/ADC2_CH2)
- new net BUCK_EN_S: U1.19 (GPIO14/ADC2_CH3)
- new net BuckPGOOD_S: R45.2, TP13.1
- new net DeployV: J1.5 (Pin_5), J1.6 (Pin_6)
- new net Switch_2: J9.1 (Pin_1), R48.1, U1.6 (GPIO1/ADC1_CH0)
Other:
- sheet Linear Actuator ports: added Fault, M1; removed none
- moved on the sheet: C3, C8

Commit message: formatting
Parts:
- C103: renamed from C8; value 0.1uF -> 100nF
- C105: renamed from C5; value 0.1uF -> 100nF
- C106: renamed from C6; value 0.1uF -> 100nF
- C109: renamed from C10; value 0.1uF -> 100nF
- C110: renamed from C3; value 0.1uF -> 100nF
- C111: renamed from C11; value 0.1uF -> 100nF
- C114: renamed from C45; value 0.1uF -> 100nF
- H101: renamed from H1; now left out of the parts list
- H102: renamed from H2; now left out of the parts list
- H103: renamed from H3; now left out of the parts list
- H104: renamed from H4; now left out of the parts list
- L101: renamed from L1; value 2.0nH -> 2nH
- LED101: renamed from LED1; value GREEN_LED -> LED_GREEN
- LED102: renamed from LED2; value GREEN_LED -> LED_GREEN
- LED103: renamed from LED3; value ORANGE_LED -> LED_ORANGE
- LED104: renamed from LED4; value BLUE_LED -> LED_BLUE
- LED105: renamed from LED5; value RED_LED -> LED_RED
- R101: renamed from R1; value 10K -> 10kΩ
- R102: renamed from R2; value 470 -> 470Ω
- R103: renamed from R5; value 1k -> 1kΩ
- R104: renamed from R18; value 1k -> 1kΩ
- R105: renamed from R3; value 10K -> 10kΩ
- R106: renamed from R4; value 470 -> 470Ω
- R107: renamed from R6; value 499R -> 499Ω
- R108: renamed from R7; value 3k -> 3kΩ
- R109: renamed from R49; value 10k -> 10kΩ
- R110: renamed from R36; value 1.5k -> 1.5kΩ
- R111: renamed from R37; value 470 -> 470Ω
- R112: renamed from R48; value 10k -> 10kΩ
- R113: renamed from R34; value 18k -> 18kΩ
- R114: renamed from R45; value 18k -> 18kΩ
- TP101: renamed from TP9; now left out of the parts list
- TP102: renamed from TP10; now left out of the parts list
- TP103: renamed from TP25; now left out of the parts list
- TP104: renamed from TP26; now left out of the parts list
- TP105: renamed from TP27; now left out of the parts list
- TP106: renamed from TP7; now left out of the parts list
- TP107: renamed from TP14; now left out of the parts list
- TP108: renamed from TP11; now left out of the parts list
- TP109: renamed from TP13; now left out of the parts list
- renumbered C1 to C101, C2 to C102, C4 to C104, C7 to C107, C9 to C108, C13 to C112, C14 to C113, J11 to J101, J1 to J102, J10 to J103, J9 to J104, J7 to J105, L2 to L102, U1 to U101, Y1 to Y101
Other:
- moved on the sheet: C103, C110, C114, J102, J103, J104, J105, R109, R110, R111, R112, R113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

Commit message: feat: Post Jack review
Changed buck inductors to be wuerth. Reduced board footprint. Incorporated review feedback
Parts:
- removed TP103, TP104, TP105, TP106: TestPoint, TestPoint:TestPoint_Pad_D1.0mm, symbol Connector:TestPoint
- LED102: Name (none) -> CAN_TX
- LED103: Name (none) -> CAN_RX
Connections:
- net BUS_VMON: now also U101.6 (GPIO1/ADC1_CH0); no longer U101.24 (GPIO18/ADC2_CH7/DAC_1)
- net DIR/BPHASE: now also U101.45 (MTDO/JTAG/GPIO40); no longer U101.39 (GPIO34)
- net NENBL/AENBL: now also U101.40 (GPIO35); no longer U101.41 (GPIO36)
- net NSLEEP: now also U101.24 (GPIO18/ADC2_CH7/DAC_1); no longer U101.38 (GPIO33)
- net STEP/BENBL: now also U101.39 (GPIO34); no longer U101.40 (GPIO35)
- net Switch_1: now also U101.38 (GPIO33); no longer U101.45 (MTDO/JTAG/GPIO40)
- net Switch_2: now also U101.41 (GPIO36); no longer U101.6 (GPIO1/ADC1_CH0)
